File: nrf24 leonardo prototype.sch (EAGLE design)
At the start: 5 parts

Commit message: Update
Just moved a few things
Other:
- note added: "LEONARDO NRF24 SHIELD REV1.0 JORDAN JONES July 2015"
Changed lines of the file:
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@@
 <sheet>
 <plain>
+<text x="-88.9" y="-20.32" size="1.778" layer="91">LEONARDO NRF24 SHIELD
+REV1.0
+JORDAN JONES
+July 2015</text>
 </plain>
 <instances>
@@
 </schematic>
 </drawing>
+<compatibility>
+<note version="6.3" minversion="6.2.2" severity="warning">
+Since Version 6.2.2 text objects can contain more than one line,
+which will not be processed correctly with this version.
+</note>
+</compatibility>
 </eagle>
